File: pcb/release/isa-sdcard.kicad_pcb (KiCad board)
At the start: 4 copper layers, 104.4 x 82.7 mm, 51 parts, among them J1 Micro_SD_Card_Det1, J2 Bus_ISA_8bit_AB_Rev0, SW1 ADDR SEL, U1 74HC00, U10 74HC74, U11 74HC08, U12 74HC04, U13 74HC74, U16 AMS1117-3.3, U2 74HCT32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

Commit message: Adding delays and improving bracket
Parts:
- removed the REF** at (83.3, 74.2)
- added C15: 0.1uF, Capacitor_SMD:C_0805_2012Metric, F.Cu at (128.5, 86.5)
- added C7: 0.1uF, Capacitor_SMD:C_0805_2012Metric, F.Cu at (150.1, 86.5)
- added R5: 10k, Resistor_SMD:R_0805_2012Metric, F.Cu at (150.1, 90.3)
- added R6: 10k, Resistor_SMD:R_0805_2012Metric, F.Cu at (128.5, 90.3)
- added REF**: OSHW-Logo2_7.3x6mm_SilkScreen, Symbol:OSHW-Logo2_7.3x6mm_SilkScreen, F.Cu at (82.3, 87.4)
- moved REF** 19.9 mm to (82.0, 75.9), turned to 90 degrees
Routing:
- net ~{SDCS_SET}: track 27.6 -> 54.2 mm, vias 2 -> 3
- net ~{SDOUT_RESET}: track 9.24 -> 30.2 mm, vias 0 -> 2
- net ~{SER_RD_AND_PULSE}: track 100.5 -> 105.3 mm
- net GND: track 120.6 -> 124.9 mm, vias 39 -> 41
- net VCC: track 171.0 -> 174.6 mm, vias 41 -> 43
- net ~{SER_WR}: track 123.4 -> 125.2 mm
- net Net-(U13B-~{Q}): track 59.3 -> 58.0 mm
- net ~{PORTSEL}: track 88.9 -> 89.8 mm
- net ~{SDOUT_SET}: track 11.7 -> 12.4 mm
Other:
- board text added: "https://github.com/ifilot/slot-otter"
- board text added: "rev2"
- board text removed: "rev1"

Commit message: Removing delay lines
Parts:
- removed C15, C7: 0.1uF, Capacitor_SMD:C_0805_2012Metric
- removed R5, R6: 10k, Resistor_SMD:R_0805_2012Metric
- removed the REF** at (82.3, 87.4)
- added REF**: OSHW-Logo2_9.8x8mm_SilkScreen, Symbol:OSHW-Logo2_9.8x8mm_SilkScreen, F.Cu at (83.3, 74.2)
- moved REF** 19.4 mm to (96.5, 63.0), turned to 0 degrees
- moved X1 17.0 mm to (92.2, 54.3), turned to 0 degrees
Routing:
- net ~{SDCS_SET}: track 54.2 -> 27.6 mm, vias 3 -> 2
- net ~{SDOUT_RESET}: track 30.2 -> 9.24 mm, vias 2 -> 0
- net ~{SER_RD_AND_PULSE}: track 105.3 -> 100.5 mm
- net GND: track 124.9 -> 120.6 mm, vias 41 -> 39
- net VCC: track 174.6 -> 171.0 mm, vias 43 -> 41
- net ~{SER_WR}: track 125.2 -> 123.4 mm
- net 16MHz: track 68.4 -> 70.0 mm
- net Net-(U13B-~{Q}): track 58.0 -> 59.3 mm
- net ~{PORTSEL}: track 89.8 -> 88.9 mm
- net ~{SDOUT_SET}: track 12.4 -> 11.7 mm
