File: pcb/release/isa-sdcard.kicad_sch (KiCad schematic)
At the start: 48 parts, among them J1 Micro_SD_Card_Det1, J2 Bus_ISA_8bit_AB_Rev0, SW1 ADDR SEL, U1 74HC00, U10 74HC74, U11 74HC08, U12 74HC04, U13 74HC74, U16 AMS1117-3.3, U2 74HCT32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

Commit message: Adding JLCPCB numbers
Parts:
- C1, C11, C12, C13, C14, C2, C3, C4, C5, C6, C8, C9: LCSC (none) -> C126469; LCSC Part # C126469 -> (none)
- C10: value 100n -> 0.1uF; LCSC (none) -> C126469
- C23: LCSC (none) -> C309030; LCSC Part # C309030 -> (none)
- D1, D2, D3: LCSC (none) -> C84256
- J1: LCSC (none) -> C381082; LCSC Part # C381082 -> (none)
- R1: LCSC (none) -> C5159708; LCSC Part # C5159708 -> (none)
- R10, R11, R8, R9: LCSC (none) -> C407459; LCSC Part # C407459 -> (none)
- R2, R3, R4: LCSC (none) -> C17540
- RN1, RN3: LCSC (none) -> C29718
- U1, U5: LCSC (none) -> C699445; LCSC Part # C699445 -> (none)
- U10, U13: LCSC (none) -> C6762
- U11: LCSC (none) -> C5593
- U12: LCSC (none) -> C5590
- U16: LCSC (none) -> C5346136; LCSC Part # C5346136 -> (none)
- U2: LCSC (none) -> C5985
- U21: LCSC (none) -> C7494906
- U21: LCSC (none) -> C7494906; LCSC Part # C7494906 -> (none)
- U3: LCSC (none) -> C545677
- U4: LCSC (none) -> C338758; LCSC Part # C338758 -> (none)
- U6: LCSC (none) -> C5613; LCSC Part # C5613 -> (none)
- U7: LCSC (none) -> C5947; LCSC Part # C5947 -> (none)
- U8: LCSC (none) -> C2649422
- U9: LCSC (none) -> C5979
