File: pcb/cpld/cpld.kicad_sch (KiCad schematic)
At the start: 31 parts, among them J1 Micro_SD_Card_Det1, J2 Bus_ISA_8bit_AB_Rev0, J3 Atmel-JTAG-10, SW1 ADDR SEL, U1 ATF1504AS-xJx44, U2 AMS1117-3.3, U3 74LVC125, U4 74HCT688, X1 16MHz

Commit message: Prepare Slot-otter v1.1.0 with CPLD revision 1.0 hardware (#7)
* Incrementing version number

* Restore DOS CRLF line endings in updated source files (#5)

* Expanding explanation and polishing settings interface

* Increasing maximum number of files per folder

* Fixing files for MSDOS

* Initial commit SD-CARD write routines

* Improving commenting and routines

* Tuning write cycles

* Improving schematic, improving sd commands and making cross-compilation more convenient

* Adding JLCPCB numbers

* Implementing folder creation

* Refactoring otternav and initial commit copying from HD to SD

* Refining CPLD card

* Initial commit DRIVER

* Working RW driver

* Consolidation step

* Consolidating for v1.0.0 of the driver

* Adding CPLD logic

* Redesigning CPLD PCB

* Final tweaks CPLD

* Refactoring for release

* Improving README.md

* Keep CPLD fabrication archive in sync with Gerber exports

* Prepare Slot-otter 1.1.0 hardware and software release

* Display README hardware renders side by side

* Show Nightwatch screenshot in the user guide
Parts:
- removed J3: Atmel-JTAG-10, Connector_IDC:IDC-Header_2x05_P2.54mm_Vertical, symbol atf1504_plcc44_breakout:Atmel-JTAG-10
- removed TP1: ~{CS}, TestPoint:TestPoint_Loop_D2.54mm_Drill1.5mm_Beaded, symbol Connector:TestPoint_Probe
- removed TP2: CLK, TestPoint:TestPoint_Loop_D2.54mm_Drill1.5mm_Beaded, symbol Connector:TestPoint_Probe
- removed TP3: MOSI, TestPoint:TestPoint_Loop_D2.54mm_Drill1.5mm_Beaded, symbol Connector:TestPoint_Probe
- removed TP4: MISO, TestPoint:TestPoint_Loop_D2.54mm_Drill1.5mm_Beaded, symbol Connector:TestPoint_Probe
- removed TP5, TP6: GND, TestPoint:TestPoint_Loop_D2.54mm_Drill1.5mm_Beaded, symbol Connector:TestPoint_Probe
- added SYM1: (no value), components:slototter-logo-v2, symbol logo:LOGO
- added SYM2: (no value), Symbol:OSHW-Logo_11.4x12mm_SilkScreen, symbol logo:LOGO
- J1: symbol Connector:Micro_SD_Card_Det1 -> slototter-connectors:Micro_SD_Card_Det1
- J2: symbol Connector:Bus_ISA_8bit_AB_Rev0 -> slototter-connectors:Bus_ISA_8bit_AB_Rev0
- U1: value ATF1504AS-xJx44 -> ATF1504AS
- U3: footprint (none) -> Package_SO:TSSOP-14_4.4x5mm_P0.65mm
Connections:
- net 16MHz: now also U1.2 (I/OE2/GCLK2); no longer U1.43 (I/GCLK1)
- net A0: now also U1.17 (I/O); no longer U1.18 (I/O)
- net CLK: now also U1.4 (I/O); no longer U1.28 (I/O)
- net DB0: now also U1.21 (I/O); no longer U1.29 (I/O)
- net DB1: now also U1.25 (I/O/PD2); no longer U1.31 (I/O)
- net DB2: now also U1.26 (I/O); no longer U1.33 (I/O)
- net DB3: now also U1.27 (I/O); no longer U1.34 (I/O)
- net DB4: now also U1.28 (I/O); no longer U1.36 (I/O)
- net DB5: now also U1.29 (I/O); no longer U1.37 (I/O)
- net DB6: now also U1.31 (I/O); no longer U1.39 (I/O)
- net DB7: now also U1.33 (I/O); no longer U1.40 (I/O)
- net MISO: now also U1.12 (I/O); no longer U1.25 (I/O/PD2)
- net MOSI: now also U1.6 (I/O); no longer U1.24 (I/O)
- net ~{CS}: now also U1.40 (I/O); no longer U1.27 (I/O)
- net ~{PORTSEL}: now also U1.9 (I/O); no longer U1.44 (I/OE1)
- net ~{RD}: now also U1.18 (I/O); no longer U1.16 (I/O)
- net ~{WR}: now also U1.20 (I/O); no longer U1.17 (I/O)
- net MISO_PULL: now reaches R1.2
- net MISO_PULL: now also U1.24 (I/O); no longer U1.26 (I/O)
- net TCK: no longer names the net of U1.32 (I/O/TCK)
- net TDI: no longer names the net of U1.7 (I/O/TDI)
- net TDO: no longer names the net of U1.38 (I/O/TDO)
- net TMS: no longer names the net of U1.13 (I/O/TMS)
- no-connect marks 53 -> 57
Other:
- title: ISA-TO-SDCARD -> Slot-otter CPLD
- moved on the sheet: C1, C2, C3, C4, C5, C6, C7, H1, H2, J1, J2, R1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
