File: pcb/cpld/cpld.kicad_sch (KiCad schematic)
At the start: 31 parts, among them J1 Micro_SD_Card_Det1, J2 Bus_ISA_8bit_AB_Rev0, J3 Atmel-JTAG-10, SW1 ADDR SEL, U1 ATF1504AS-xJx44, U2 AMS1117-3.3, U3 74LVC125, U4 74HCT688, X1 16MHz

Commit message: Redesigning CPLD PCB
Parts:
- removed J3: Atmel-JTAG-10, Connector_IDC:IDC-Header_2x05_P2.54mm_Vertical, symbol atf1504_plcc44_breakout:Atmel-JTAG-10
- removed TP1: ~{CS}, TestPoint:TestPoint_Loop_D2.54mm_Drill1.5mm_Beaded, symbol Connector:TestPoint_Probe
- removed TP2: CLK, TestPoint:TestPoint_Loop_D2.54mm_Drill1.5mm_Beaded, symbol Connector:TestPoint_Probe
- removed TP3: MOSI, TestPoint:TestPoint_Loop_D2.54mm_Drill1.5mm_Beaded, symbol Connector:TestPoint_Probe
- removed TP4: MISO, TestPoint:TestPoint_Loop_D2.54mm_Drill1.5mm_Beaded, symbol Connector:TestPoint_Probe
- removed TP5, TP6: GND, TestPoint:TestPoint_Loop_D2.54mm_Drill1.5mm_Beaded, symbol Connector:TestPoint_Probe
- added SYM1: (no value), components:slototter-logo-v2, symbol logo:LOGO
- U3: footprint (none) -> Package_SO:TSSOP-14_4.4x5mm_P0.65mm
Connections:
- net 16MHz: now also U1.2 (I/OE2/GCLK2); no longer U1.43 (I/GCLK1)
- net A0: now also U1.17 (I/O); no longer U1.18 (I/O)
- net CLK: now also U1.4 (I/O); no longer U1.28 (I/O)
- net DB0: now also U1.21 (I/O); no longer U1.29 (I/O)
- net DB1: now also U1.25 (I/O/PD2); no longer U1.31 (I/O)
- net DB2: now also U1.26 (I/O); no longer U1.33 (I/O)
- net DB3: now also U1.27 (I/O); no longer U1.34 (I/O)
- net DB4: now also U1.28 (I/O); no longer U1.36 (I/O)
- net DB5: now also U1.29 (I/O); no longer U1.37 (I/O)
- net DB6: now also U1.31 (I/O); no longer U1.39 (I/O)
- net DB7: now also U1.33 (I/O); no longer U1.40 (I/O)
- net MISO: now also U1.12 (I/O); no longer U1.25 (I/O/PD2)
- net MOSI: now also U1.6 (I/O); no longer U1.24 (I/O)
- net ~{CS}: now also U1.40 (I/O); no longer U1.27 (I/O)
- net ~{PORTSEL}: now also U1.9 (I/O); no longer U1.44 (I/OE1)
- net ~{RD}: now also U1.18 (I/O); no longer U1.16 (I/O)
- net ~{WR}: now also U1.20 (I/O); no longer U1.17 (I/O)
- net MISO_PULL: now reaches R1.2
- net MISO_PULL: now also U1.24 (I/O); no longer U1.26 (I/O)
- net TCK: no longer names the net of U1.32 (I/O/TCK)
- net TDI: no longer names the net of U1.7 (I/O/TDI)
- net TDO: no longer names the net of U1.38 (I/O/TDO)
- net TMS: no longer names the net of U1.13 (I/O/TMS)
- no-connect marks 53 -> 57
Other:
- moved on the sheet: C1, C2, C3, C4, C5, C6, C7, H1, H2, J1, J2, R1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

Commit message: Final tweaks CPLD
Parts:
- added SYM2: (no value), Symbol:OSHW-Logo_11.4x12mm_SilkScreen, symbol logo:LOGO
- U1: value ATF1504AS-xJx44 -> ATF1504AS
Changed lines of the file:
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@@
 			)
 		)
-		(property "Value" "ATF1504AS-xJx44"
+		(property "Value" "ATF1504AS"
 			(at 46.5933 24.13 0)
 			(show_name no)
@@
 					(unit 1)
 				)
+			)
+		)
+	)
+	(symbol
+		(lib_id "logo:LOGO")
+		(at 191.77 162.56 0)
+		(unit 1)
+		(body_style 1)
+		(exclude_from_sim no)
+		(in_bom yes)
+		(on_board yes)
+		(in_pos_files yes)
+		(dnp no)
+		(fields_autoplaced yes)
+		(property "Reference" "SYM2"
+			(at 194.31 162.5599 0)
+			(show_name no)
+			(do_not_autoplace no)
+			(effects
+				(font
+					(size 1.27 1.27)
+				)
+				(justify left)
+			)
+		)
+		(property "Value" ""
+			(at 191.77 162.56 0)
+			(show_name no)
+			(do_not_autoplace no)
+			(effects
+				(font
+					(size 1.27 1.27)
+				)
+			)
+		)
+		(property "Footprint" "Symbol:OSHW-Logo_11.4x12mm_SilkScreen"
+			(at 191.77 162.56 0)
+			(hide yes)
+			(show_name no)
+			(do_not_autoplace no)
+			(effects
+				(font
+					(size 1.27 1.27)
+				)
+			)
+		)
+		(property "Datasheet" ""
+			(at 191.77 162.56 0)
+			(hide yes)
+			(show_name no)
+			(do_not_autoplace no)
+			(effects
+				(font
+					(size 1.27 1.27)
+				)
+			)
+		)
+		(property "Description" ""
+			(at 191.77 162.56 0)
+			(hide yes)
+			(show_name no)
+			(do_not_autoplace no)
+			(effects
+				(font
+					(size 1.27 1.27)
+				)
+			)
+		)
+		(instances
+			(project "cpld"
+				(path "/075aea89-321c-44ba-b0b1-8b82a6b1f518"
+					(reference "SYM2")
+					(unit 1)
+				)

Commit message: Refactoring for release
Parts:
- J1: symbol Connector:Micro_SD_Card_Det1 -> slototter-connectors:Micro_SD_Card_Det1
- J2: symbol Connector:Bus_ISA_8bit_AB_Rev0 -> slototter-connectors:Bus_ISA_8bit_AB_Rev0
- SYM1, SYM2: now left out of the parts list
Other:
- title: ISA-TO-SDCARD -> Slot-otter CPLD
Changed lines of the file:
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@@
 	(paper "A4")
 	(title_block
-		(title "ISA-TO-SDCARD")
-		(date "2025-08-17")
-		(rev "rev0")
+		(title "Slot-otter CPLD")
+		(date "2026-10-16")
+		(rev "1.0")
+		(comment 1 "Hardware: CERN-OHL-S-2.0; source: github.com/ifilot/slot-otter")
 	)
 	(text "SCK"
@@
 		(body_style 1)
 		(exclude_from_sim no)
-		(in_bom yes)
+		(in_bom no)
 		(on_board yes)
-		(in_pos_files yes)
+		(in_pos_files no)
 		(dnp no)
 		(fields_autoplaced yes)
@@
 	)
 	(symbol
-		(lib_id "Connector:Micro_SD_Card_Det1")
+		(lib_id "slototter-connectors:Micro_SD_Card_Det1")
 		(at 252.73 143.51 0)
 		(unit 1)
@@
 			)
 		)
-		(property "Datasheet" "http://ww1.microchip.com/downloads/en/DeviceDoc/Atmel-0995-CPLD-ATF1502AS(L)-Datasheet.pdf"
+		(property "Datasheet" "https://ww1.microchip.com/downloads/en/DeviceDoc/ATF1504AS(L)-5V-64-Macrocell-CPLD-Data-Sheet-20006580A.pdf"
 			(at 40.64 12.7 0)
 			(hide yes)
@@
 	)
 	(symbol
-		(lib_id "Connector:Bus_ISA_8bit_AB_Rev0")
+		(lib_id "slototter-connectors:Bus_ISA_8bit_AB_Rev0")
 		(at 247.65 62.23 0)
 		(unit 1)
@@
 		(body_style 1)
 		(exclude_from_sim no)
-		(in_bom yes)
+		(in_bom no)
 		(on_board yes)
-		(in_pos_files yes)
+		(in_pos_files no)
 		(dnp no)
 		(fields_autoplaced yes)

Commit message: Revising CPLD board and adding OSHWA certification
Parts:
- added SYM3: oshw-certificate, components:oshwa_h15, symbol logo:LOGO
- added SYM4: kicad-logo, Symbol:KiCad-Logo2_5mm_SilkScreen, symbol logo:LOGO
- SYM1: value (none) -> otterlogo; footprint components:slototter-logo-v2 -> components:slototter-logo-v2_h12
- SYM2: value (none) -> oshw-logo; footprint Symbol:OSHW-Logo_11.4x12mm_SilkScreen -> Symbol:OSHW-Logo_7.5x8mm_SilkScreen
Other:
- moved on the sheet: SYM1, SYM2
Changed lines of the file:
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@@
 	(symbol
 		(lib_id "logo:LOGO")
-		(at 180.34 162.56 0)
+		(at 180.34 153.67 0)
 		(unit 1)
 		(body_style 1)
@@
 		(in_pos_files no)
 		(dnp no)
-		(fields_autoplaced yes)
 		(property "Reference" "SYM1"
-			(at 182.88 162.5599 0)
+			(at 182.88 153.6699 0)
 			(show_name no)
 			(do_not_autoplace no)
@@
 			)
 		)
-		(property "Value" ""
-			(at 180.34 162.56 0)
+		(property "Value" "otterlogo"
+			(at 180.594 155.956 0)
 			(show_name no)
 			(do_not_autoplace no)
@@
 			)
 		)
-		(property "Footprint" "components:slototter-logo-v2"
-			(at 180.34 162.56 0)
+		(property "Footprint" "components:slototter-logo-v2_h12"
+			(at 180.34 153.67 0)
 			(hide yes)
 			(show_name no)
@@
 		)
 		(property "Datasheet" ""
-			(at 180.34 162.56 0)
+			(at 180.34 153.67 0)
 			(hide yes)
 			(show_name no)
@@
 		)
 		(property "Description" ""
-			(at 180.34 162.56 0)
+			(at 180.34 153.67 0)
 			(hide yes)
 			(show_name no)
@@
 	)
 	(symbol
+		(lib_id "logo:LOGO")
+		(at 199.39 153.67 0)
+		(unit 1)
+		(body_style 1)
+		(exclude_from_sim no)
+		(in_bom no)
+		(on_board yes)
+		(in_pos_files no)
+		(dnp no)
+		(property "Reference" "SYM3"
+			(at 201.93 153.6699 0)
+			(show_name no)
+			(do_not_autoplace no)
+			(effects
+				(font
+					(size 1.27 1.27)
+				)
+				(justify left)
+			)
+		)
+		(property "Value" "oshw-certificate"
+			(at 199.39 155.956 0)
+			(show_name no)
+			(do_not_autoplace no)
+			(effects
+				(font
+					(size 1.27 1.27)
+				)
+			)
+		)
+		(property "Footprint" "components:oshwa_h15"
+			(at 199.39 153.67 0)
+			(hide yes)
+			(show_name no)
+			(do_not_autoplace no)
+			(effects
+				(font
+					(size 1.27 1.27)
+				)
+			)
+		)
+		(property "Datasheet" ""
+			(at 199.39 153.67 0)
+			(hide yes)
+			(show_name no)
+			(do_not_autoplace no)
+			(effects
+				(font
+					(size 1.27 1.27)
+				)
+			)
+		)
+		(property "Description" ""
+			(at 199.39 153.67 0)
+			(hide yes)
+			(show_name no)
+			(do_not_autoplace no)
+			(effects
+				(font
+					(size 1.27 1.27)
+				)
+			)
+		)
+		(instances
+			(project "cpld"
+				(path "/075aea89-321c-44ba-b0b1-8b82a6b1f518"
+					(reference "SYM3")
+					(unit 1)
+				)
+			)
+		)
+	)
+	(symbol
 		(lib_id "Device:R_Pack04_Split")
 		(at 62.23 172.72 0)
@@
 	)
 	(symbol
+		(lib_id "logo:LOGO")
+		(at 199.39 160.02 0)
+		(unit 1)
+		(body_style 1)
+		(exclude_from_sim no)
+		(in_bom no)
+		(on_board yes)
+		(in_pos_files no)
+		(dnp no)
+		(property "Reference" "SYM4"
+			(at 201.93 160.0199 0)
+			(show_name no)
+			(do_not_autoplace no)
+			(effects
+				(font
+					(size 1.27 1.27)
+				)
+				(justify left)
+			)
+		)
+		(property "Value" "kicad-logo"
+			(at 199.39 162.306 0)
+			(show_name no)
+			(do_not_autoplace no)
+			(effects
+				(font
+					(size 1.27 1.27)
+				)
+			)
+		)
+		(property "Footprint" "Symbol:KiCad-Logo2_5mm_SilkScreen"
+			(at 199.39 160.02 0)
+			(hide yes)
+			(show_name no)
+			(do_not_autoplace no)
+			(effects
+				(font
+					(size 1.27 1.27)
+				)
+			)
+		)
+		(property "Datasheet" ""
+			(at 199.39 160.02 0)
+			(hide yes)
+			(show_name no)
+			(do_not_autoplace no)
+			(effects
+				(font
+					(size 1.27 1.27)
+				)
+			)
+		)
+		(property "Description" ""
+			(at 199.39 160.02 0)
+			(hide yes)
+			(show_name no)
+			(do_not_autoplace no)
+			(effects
+				(font
+					(size 1.27 1.27)
+				)
+			)
+		)
+		(instances
+			(project "cpld"
+				(path "/075aea89-321c-44ba-b0b1-8b82a6b1f518"
+					(reference "SYM4")
+					(unit 1)
+				)
+			)
+		)
+	)
+	(symbol
 		(lib_id "power:GND")
 		(at 149.86 48.26 0)
@@
 	(symbol
 		(lib_id "logo:LOGO")
-		(at 191.77 162.56 0)
+		(at 180.34 160.02 0)
 		(unit 1)
 		(body_style 1)
@@
 		(in_pos_files no)
 		(dnp no)
-		(fields_autoplaced yes)
 		(property "Reference" "SYM2"
-			(at 194.31 162.5599 0)
+			(at 182.88 160.0199 0)
 			(show_name no)
 			(do_not_autoplace no)
@@
 			)
 		)
-		(property "Value" ""
-			(at 191.77 162.56 0)
+		(property "Value" "oshw-logo"
+			(at 180.34 162.306 0)
 			(show_name no)
 			(do_not_autoplace no)
@@
 			)
 		)
-		(property "Footprint" "Symbol:OSHW-Logo_11.4x12mm_SilkScreen"
-			(at 191.77 162.56 0)
+		(property "Footprint" "Symbol:OSHW-Logo_7.5x8mm_SilkScreen"
+			(at 180.34 160.02 0)
 			(hide yes)
 			(show_name no)
@@
 		)
 		(property "Datasheet" ""
-			(at 191.77 162.56 0)
+			(at 180.34 160.02 0)
 			(hide yes)
 			(show_name no)
@@
 		)
 		(property "Description" ""
-			(at 191.77 162.56 0)
+			(at 180.34 160.02 0)
 			(hide yes)
 			(show_name no)
